Commit message: cambios mapa y lidar

File: robot.urdf (robot description, URDF)
Before this commit: robot rover_basico, 1 links, 0 joints
Links:
- added link rueda_dd, mass 0.5; collision cylinder length=0.05 radius=0.07; visual cylinder length=0.05 radius=0.07
- added link rueda_di, mass 0.5; collision cylinder length=0.05 radius=0.07; visual cylinder length=0.05 radius=0.07
- added link rueda_td, mass 0.5; collision cylinder length=0.05 radius=0.07; visual cylinder length=0.05 radius=0.07
- added link rueda_ti, mass 0.5; collision cylinder length=0.05 radius=0.07; visual cylinder length=0.05 radius=0.07
- link chasis: mass 5.0 -> 3.0; geometry collision box size=0.4 0.3 0.08; visual box size=0.4 0.3 0.08
Joints:
- added joint joint_rueda_dd: type continuous, parent chasis, child rueda_dd, origin xyz=0.15 -0.175 -0.01, axis 0 1 0
- added joint joint_rueda_di: type continuous, parent chasis, child rueda_di, origin xyz=0.15 0.175 -0.01, axis 0 1 0
- added joint joint_rueda_td: type continuous, parent chasis, child rueda_td, origin xyz=-0.15 -0.175 -0.01, axis 0 1 0
- added joint joint_rueda_ti: type continuous, parent chasis, child rueda_ti, origin xyz=-0.15 0.175 -0.01, axis 0 1 0

Commit message: lol

File: robot.urdf (robot description, URDF)
Before this commit: robot rover_basico, 5 links, 4 joints
Links:
- link chasis: mass 3.0 -> 4.0; geometry collision box size=0.35 0.30 0.06; visual box size=0.35 0.30 0.06
- link rueda_dd: geometry collision cylinder length=0.04 radius=0.055; visual cylinder length=0.04 radius=0.055
- link rueda_di: geometry collision cylinder length=0.04 radius=0.055; visual cylinder length=0.04 radius=0.055
- link rueda_td: geometry collision cylinder length=0.04 radius=0.055; visual cylinder length=0.04 radius=0.055
- link rueda_ti: geometry collision cylinder length=0.04 radius=0.055; visual cylinder length=0.04 radius=0.055
Joints:
- joint joint_rueda_dd: origin xyz=0.15 -0.175 -0.01 -> xyz=0.13 -0.17 -0.005
- joint joint_rueda_di: origin xyz=0.15 0.175 -0.01 -> xyz=0.13 0.17 -0.005
- joint joint_rueda_td: origin xyz=-0.15 -0.175 -0.01 -> xyz=-0.13 -0.17 -0.005
- joint joint_rueda_ti: origin xyz=-0.15 0.175 -0.01 -> xyz=-0.13 0.17 -0.005
